File: Avionics-Argus3-BatteryBoard.kicad_pcb (KiCad board)
At the start: 4 copper layers, 90.2 x 95.9 mm, 143 parts, among them J1 Keystone-1048, J2 Keystone-1048, J3 Keystone-1042, J4 Keystone-1042, J5 Fuel Gauge Programming Header, J6 205338-0002, J7 205338-0004, J8 282834-4, J9 522711069, Q1 SIRA99DP-T1-GE3, Q10 SIRA99DP-T1-GE3, Q11 MBT2222ADW1T1, Q12 NX3008NBKS, Q13 MBT2222ADW1T1, Q14 NX3008NBKS, Q2 IRLML2803, Q3 SIRA99DP-T1-GE3, Q4 IRLML2803, Q5 SIRA99DP-T1-GE3, Q6 IRLML2803, Q7 SIRA99DP-T1-GE3, Q8 SIRA99DP-T1-GE3, Q9 SIRA99DP-T1-GE3, U1 S-8209AAA-T8T1U, U2 S-8209AAA-T8T1U, U3 LTC4412xS6, U4 LTC4412xS6, U5 MAX17205, U6 D5V0P4UR6SO, U7 D5V0P4UR6SO

Commit message: Layout in progress
In the middle of completing layout
Parts:
- removed F5, F6: 5A, Fuse:Fuse_1206_3216Metric
- removed J3, J4: Keystone-1042, Argus-Misc:Keystone_1042
- removed R21, R22, R23: 10R, Resistor_SMD:R_2512_6332Metric
- removed TH3, TH6: 10k 3435k, Capacitor_SMD:C_0603_1608Metric
- added C14: 100n, Capacitor_SMD:C_0603_1608Metric, B.Cu at (223.7, 119.4)
- added C15: 100n, Capacitor_SMD:C_0603_1608Metric, B.Cu at (223.7, 121.9)
- added C16: 100n, Capacitor_SMD:C_0603_1608Metric, B.Cu at (223.7, 124.4)
- added C17: 10u, Capacitor_SMD:C_0603_1608Metric, B.Cu at (223.7, 126.9)
- added C18: 1u, Capacitor_SMD:C_0603_1608Metric, B.Cu at (223.7, 129.4)
- added C19: 100n, Capacitor_SMD:C_0603_1608Metric, B.Cu at (219.7, 119.4)
- added C20: 1u, Capacitor_SMD:C_0603_1608Metric, B.Cu at (219.7, 121.9)
- added C21: 4.7u, Capacitor_SMD:C_0603_1608Metric, B.Cu at (219.7, 124.4)
- added C22: 100n, Capacitor_SMD:C_0603_1608Metric, B.Cu at (219.7, 126.9)
- added C23: 12p, Capacitor_SMD:C_0603_1608Metric, B.Cu at (219.7, 129.4)
- added C24: 12p, Capacitor_SMD:C_0603_1608Metric, B.Cu at (215.7, 119.4)
- added C25: 100n, Capacitor_SMD:C_0603_1608Metric, B.Cu at (215.7, 121.9)
- added C26: 10u, Capacitor_SMD:C_0805_2012Metric, B.Cu at (214.4, 95.5)
- added C27: 1u, Capacitor_SMD:C_0603_1608Metric, B.Cu at (218.7, 95.3)
- added C28: 22u, Capacitor_SMD:C_0805_2012Metric, B.Cu at (214.4, 98.6)
- added D7: GRN, LED_SMD:LED_0603_1608Metric, B.Cu at (211.7, 125.7)
- added IC1: STM32U375CET6, Argus-Misc:QFP50P900X900X160-48N, B.Cu at (144.8, 66.9)
- added L1: 6.8u, Argus-Passives:ECS-MPI4040, B.Cu at (223.3, 96.9)
- added Q15: IRLML2803, Package_TO_SOT_SMD:SOT-23, B.Cu at (207.9, 105.8)
- added Q16: IRLML2803, Package_TO_SOT_SMD:SOT-23, B.Cu at (214.8, 105.8)
- added Q17: IRLML2803, Package_TO_SOT_SMD:SOT-23, B.Cu at (214.8, 110.2)
- added R66: 10k, Resistor_SMD:R_0603_1608Metric, B.Cu at (215.7, 124.4)
- added R67: 120, Resistor_SMD:R_0603_1608Metric, B.Cu at (215.7, 126.9)
- added R69: NP, Resistor_SMD:R_0603_1608Metric, B.Cu at (218.7, 97.8)
- added R70: 2.7k, Resistor_SMD:R_0603_1608Metric, B.Cu at (218.7, 100.3)
- added R71: 10k, Resistor_SMD:R_0603_1608Metric, B.Cu at (217.7, 133.9)
- added R72: R, Resistor_SMD:R_0603_1608Metric, B.Cu at (205.2, 83.8)
- added R73: R, Resistor_SMD:R_0603_1608Metric, B.Cu at (205.2, 86.3)
- added R74: R, Resistor_SMD:R_0603_1608Metric, B.Cu at (205.2, 88.8)
- added R75: R, Resistor_SMD:R_0603_1608Metric, B.Cu at (205.2, 91.3)
- added R76: 10k, Resistor_SMD:R_0603_1608Metric, B.Cu at (223.7, 133.9)
- added R77: 10k, Resistor_SMD:R_0603_1608Metric, B.Cu at (223.7, 136.4)
- added U10: SN74LVC32AD, Argus-Misc:D14, B.Cu at (221.7, 108.8)
- added U6: TPS62111RSA, Package_DFN_QFN:Texas_RSA_VQFN-16-1EP_4x4mm_P0.65mm_EP2.7x2.7mm, B.Cu at (210.2, 121.3)
- added U8: TCAN330, Package_TO_SOT_SMD:SOT-23-8, B.Cu at (211.9, 89.5)
- added Y1: Crystal_GND24, Crystal:Crystal_SMD_3225-4Pin_3.2x2.5mm, B.Cu at (211.9, 84.8)
- R45, R46: value 30k -> 20k
- TH1: moved to F.Cu
- moved TH2 19.1 mm to (164.6, 107.5)
- moved R15 0.18 mm to (129.5, 67.1)
- moved F3 0.14 mm to (182.0, 73.6)
- moved R17 0.13 mm to (162.3, 67.0)
- moved R16 0.07 mm to (145.8, 67.2)
- moved TH1 0.06 mm to (164.6, 126.6), turned to 90 degrees
Connections:
- net /Battery Bus Detection/BATT_P renamed VIN
- J9 pad 1: /Interfaces/HEATER_ENABLE -> /MCU_Subsystem/CAN_H
- J9 pad 10: +3V3 -> GND
- J9 pad 2: /Interfaces/HEATER1_ON -> /MCU_Subsystem/CAN_L
- J9 pad 3: /Interfaces/HEATER0_ON -> GND
- J9 pad 4: /Interfaces/ALERT -> GND
- J9 pad 5: /Interfaces/SDA_BUS -> GND
- J9 pad 6: /Interfaces/SCL_BUS -> GND
- J9 pad 9: +3V3 -> GND
- Q11 pad 1: /Interfaces/SCL_BUS -> /Battery Monitor/SCL_FUEL
- Q11 pad 3: /Interfaces/SCL_BUS -> /Battery Monitor/SCL_FUEL
- Q13 pad 1: /Interfaces/SDA_BUS -> /Battery Monitor/SDA_FUEL
- Q13 pad 3: /Interfaces/SDA_BUS -> /Battery Monitor/SDA_FUEL
- Q7 pad 4: /Battery Bus Detection/CHARGE_EN -> Net-(Q15-D)
- R11 pad 2: /Interfaces/HEATER0_ON -> /Battery Temperature Protection/BatteryHeater/ENABLE
- R12 pad 2: /Interfaces/HEATER0_ON -> /Battery Temperature Protection/BatteryHeater/ENABLE
- R24 pad 2: /Interfaces/HEATER1_ON -> /Battery Temperature Protection/BatteryHeater1/ENABLE
- R25 pad 2: /Interfaces/HEATER1_ON -> /Battery Temperature Protection/BatteryHeater1/ENABLE
- R37 pad 1: +3V3 -> +3.3V
- R38 pad 2: /Battery Bus Detection/CHARGE_EN -> Net-(Q15-D)
- R40 pad 1: +3V3 -> +3.3V
- R44 pad 2: /Interfaces/ALERT -> /Battery Monitor/ALERT
- R47 pad 1: /Interfaces/ALERT -> /Battery Monitor/ALERT
- R51 pad 1: /Interfaces/ALERT -> /Battery Monitor/ALERT
- R64 pad 2: /Interfaces/SCL_BUS -> /Battery Monitor/SCL_FUEL
- R65 pad 2: /Interfaces/SDA_BUS -> /Battery Monitor/SDA_FUEL
- R7 pad 2: /Interfaces/HEATER_ENABLE -> Net-(U10-2Y)
- R8 pad 2: /Interfaces/HEATER_ENABLE -> Net-(U10-2Y)
- TH2 pad 2: Net-(TH2-Pad2) -> SYSTEM_VSS
- TH5 pad 2: Net-(TH5-Pad2) -> SYSTEM_VSS
Routing:
- net Net-(TH2-Pad2): track 17.6 -> 0.00 mm
- net Net-(TH1-Pad2): track 2.79 -> 17.6 mm, vias 1 -> 0
- net Net-(R22-Pad1): track 9.96 -> 0.00 mm
- net Net-(R21-Pad1): track 9.96 -> 0.00 mm
- net Net-(J3-NEG): track 4.00 -> 0.00 mm
- net Net-(TH5-Pad2): track 2.79 -> 0.00 mm, vias 1 -> 0
- net Net-(U5-AIN2): track 72.6 -> 73.4 mm
- net /Interfaces/SDA_BUS: vias 2 -> 0
- net /Interfaces/SCL_BUS: vias 2 -> 0
- net /Interfaces/HEATER0_ON: vias 2 -> 0
- net /Interfaces/ALERT: vias 2 -> 0
- net /Battery Temperature Protection/BatteryHeater/V_HEATER: vias 9 -> 7
- net /Battery Temperature Protection/BatteryHeater/ENABLE: vias 0 -> 2
- net /Battery Monitor/SDA_FUEL: vias 0 -> 2
- net /Battery Monitor/SCL_FUEL: vias 0 -> 2
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- added copper zone on B.Cu, net (none)
- removed copper zone on B.Cu, net Net-(J3-NEG)
- removed copper zone on B.Cu, net Net-(J4-POS)

Commit message: schematic wip
Parts:
- removed the C14 at (110.1, 93.3)
- removed R34, R35, R36: 10R, Resistor_SMD:R_2512_6332Metric
- removed the U6 at (111.2, 100.2)
- removed U7: D5V0P4UR6SO, Package_TO_SOT_SMD:SOT-23-6
- C17: footprint Capacitor_SMD:C_0603_1608Metric -> Capacitor_SMD:C_0805_2012Metric
- moved U10 113.5 mm to (115.8, 68.1)
- moved C17 109.3 mm to (138.4, 58.6)
- moved C15 105.0 mm to (137.0, 62.7)
- moved C18 99.0 mm to (150.6, 62.7)
- moved C25 99.0 mm to (132.1, 69.0), turned to 0 degrees
- moved C16 97.9 mm to (140.5, 72.8), turned to -90 degrees
- moved C14 97.1 mm to (147.4, 59.3), turned to 90 degrees
- moved R66 96.8 mm to (144.7, 58.6), turned to -90 degrees
- moved L1 95.6 mm to (132.6, 127.0)
- moved C21 92.9 mm to (142.1, 73.5), turned to -90 degrees
- moved C23 92.0 mm to (154.9, 64.2), turned to 0 degrees
- moved C22 91.5 mm to (151.5, 66.0), turned to 0 degrees
- moved R69 90.3 mm to (130.5, 117.4), turned to -90 degrees
- moved C28 89.9 mm to (129.1, 126.9), turned to 90 degrees
- moved C26 89.8 mm to (128.9, 122.8), turned to -90 degrees
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Connections:
- R54 pad 1: +3V3 -> +3.3V
- R55 pad 1: +3V3 -> +3.3V
- R59 pad 1: +3V3 -> +3.3V
- R60 pad 1: +3V3 -> +3.3V
- R75 pad 2: Net-(R75-Pad2) -> /Battery Monitor/HW_HEATER0_ON
Routing:
- net /Interfaces/ALERT: track 84.4 -> 0.00 mm
- net /Battery Monitor/ALERT: track 0.00 -> 77.1 mm, vias 2 -> 1
- net /Interfaces/SCL_BUS: track 56.6 -> 0.00 mm
- net /Interfaces/SDA_BUS: track 51.7 -> 0.00 mm
- net /Battery Monitor/SCL_FUEL: track 0.00 -> 51.2 mm, vias 2 -> 1
- net /Battery Monitor/SDA_FUEL: track 0.00 -> 46.4 mm, vias 2 -> 1
- net /Interfaces/HEATER_ENABLE: track 43.9 -> 0.00 mm, vias 2 -> 0
- net Net-(U10-2Y): track 0.00 -> 35.9 mm, vias 0 -> 1
- net /Interfaces/HEATER1_ON: track 30.7 -> 0.00 mm, vias 2 -> 0
- net /Battery Temperature Protection/BatteryHeater1/ENABLE: track 0.00 -> 25.3 mm, vias 0 -> 1
- net /Interfaces/HEATER0_ON: track 23.3 -> 0.00 mm
- net +3.3V: track 0.00 -> 22.4 mm, vias 0 -> 6
- net /Battery Temperature Protection/BatteryHeater/ENABLE: track 0.00 -> 18.0 mm, vias 2 -> 1
- net GND: track 8.59 -> 23.3 mm, vias 30 -> 32
- net +3V3: track 11.8 -> 1.05 mm, vias 2 -> 0
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- added copper zone on B.Cu, net +3.3V
- added copper zone on In1.Cu, net +3.3V
- added copper zone on B.Cu, net Net-(L1-Pad1)
- removed copper zone on B.Cu, net +3V3
Other:
- board text added: "CAN_H"
- board text added: "CAN_L"
- board text removed: "3V3"
- board text removed: "ALRT"
- board text removed: "H0_ON"
- board text removed: "H1_ON"
- board text removed: "H_EN"

Commit message: finished layout
Parts:
- removed R67: 120, Resistor_SMD:R_0603_1608Metric
- added IC2: LM393WDT, Argus-Misc:SOIC127P600X175-8N, B.Cu at (100.7, 119.1)
- moved R77 122.0 mm to (116.6, 128.9)
- moved Q17 120.0 mm to (116.5, 126.4), turned to 180 degrees
- moved R76 118.2 mm to (117.9, 120.1)
- moved Q16 112.4 mm to (118.0, 122.6), turned to 0 degrees
- moved R75 111.1 mm to (98.7, 122.7)
- moved R73 109.6 mm to (99.6, 115.5)
- moved R74 108.3 mm to (102.4, 122.7)
- moved R72 107.1 mm to (102.9, 115.5)
- moved U8 60.4 mm to (124.2, 125.6), turned to -90 degrees
- moved C21 60.0 mm to (134.1, 132.9)
- moved C14 60.0 mm to (139.5, 118.7)
- moved C15 60.0 mm to (129.1, 122.2)
- moved C16 60.0 mm to (132.6, 132.3)
- moved C18 60.0 mm to (142.7, 122.2)
- moved C19 60.0 mm to (143.5, 127.3)
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Connections:
- IC1 pad 42: /Battery Monitor/SDA_FUEL -> /Battery Monitor/SCL_FUEL
- IC1 pad 43: /Battery Monitor/SCL_FUEL -> /Battery Monitor/SDA_FUEL
- J9 pad 1: /MCU_Subsystem/CAN_H -> /MCU_Subsystem/CAN_N
- J9 pad 2: /MCU_Subsystem/CAN_L -> /MCU_Subsystem/CAN_P
- R51 pad 2: +3V3 -> +3.3V
- R57 pad 1: +3V3 -> +3.3V
- R62 pad 1: +3V3 -> +3.3V
- U8 pad 6: /MCU_Subsystem/CAN_L -> /MCU_Subsystem/CAN_N
- U8 pad 7: /MCU_Subsystem/CAN_H -> /MCU_Subsystem/CAN_P
Routing:
- net Net-(IC2-IN2-): track 73.4 -> 168.7 mm, vias 2 -> 4
- net VIN: track 0.00 -> 82.3 mm, vias 19 -> 22
- net /MCU_Subsystem/CAN_N: track 0.00 -> 63.7 mm
- net /MCU_Subsystem/CAN_P: track 0.00 -> 62.8 mm
- net GND: track 23.3 -> 75.7 mm, vias 32 -> 50
- net /Battery Monitor/HW_HEATER1_ON: track 0.00 -> 50.0 mm, vias 0 -> 2
- net /Battery Monitor/HW_HEATER0_ON: track 0.00 -> 48.9 mm, vias 0 -> 2
- net Net-(IC2-IN1-): track 71.2 -> 115.2 mm, vias 2 -> 4
- net /Battery Bus Protection/MCU_CHG_DISABLE: track 0.00 -> 41.3 mm
- net /Battery Temperature Protection/HEATER_ENABLE: track 0.00 -> 37.0 mm, vias 0 -> 2
- net /Battery Temperature Protection/HEATER1_ON: track 0.00 -> 35.2 mm, vias 0 -> 2
- net /Battery Temperature Protection/MCU_ON: track 0.00 -> 34.7 mm, vias 0 -> 2
- net /Battery Temperature Protection/HEATER0_ON: track 0.00 -> 34.5 mm, vias 0 -> 2
- net /Battery Temperature Protection/BatteryHeater/ENABLE: track 18.0 -> 47.5 mm, vias 1 -> 2
- net /Battery Monitor/ALERT: track 77.1 -> 97.4 mm, vias 1 -> 2
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