File: I2CProtection.kicad_sch (KiCad schematic)
At the start: 18 parts, among them Q11 MBT2222ADW1T1, Q12 NX3008NBKS, Q13 MBT2222ADW1T1, Q14 NX3008NBKS

Commit message: schematic wip
Connections:
- net +3V3: no longer R54.1, R55.1, R59.1, R60.1
- new net +3.3V: R54.1, R55.1, R59.1, R60.1
Changed lines of the file:
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@@
 			)
 		)
-		(property "Value" "+3V3"
+		(property "Value" "+3.3V"
 			(at 172.72 48.514 0)
 			(effects
@@
 			)
 		)
-		(property "Value" "+3V3"
+		(property "Value" "+3.3V"
 			(at 130.81 48.514 0)
 			(effects

Commit message: finished layout
Connections:
- net +3V3 is gone; now on net +3.3V: R57.1, R62.1
Changed lines of the file:
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@@
 			)
 		)
-		(property "Value" "+3V3"
+		(property "Value" "+3.3V"
 			(at 162.56 82.677 0)
 			(effects
@@
 			)
 		)
-		(property "Value" "+3V3"
+		(property "Value" "+3.3V"
 			(at 120.65 82.677 0)
 			(effects
